File: pcb/drivers/drivers.kicad_pcb (KiCad board)
At the start: 4 copper layers, 88.4 x 78.3 mm, 17 parts, among them J1 Screw_Terminal_01x02, J4 Conn_01x12_Pin, J5 Conn_01x04_Pin, J6 Conn_01x04_Pin, J7 Conn_01x04_Pin

Commit message: v0.4
Other:
- board text added: "1"
- board text added: "10"
- board text added: "11"
- board text added: "12"
- board text added: "12v"
- board text added: "2"
- board text added: "3"
- board text added: "4"
- board text added: "5"
- board text added: "6"
- board text added: "7"
- board text added: "8"
- board text added: "9"
Changed lines of the file:
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@@
 		)
 		(property "Value" "Conn_01x12_Pin"
-			(at -0.000001 30.32 25)
+			(at -0.000001 30.320001 25)
 			(layer "F.Fab")
 			(effects
@@
 		(layer "Edge.Cuts")
 	)
+	(gr_text "8"
+		(at 136.5 103 0)
+		(layer "F.SilkS")
+		(effects
+			(font
+				(size 1 1)
+				(thickness 0.1)
+			)
+			(justify left bottom)
+		)
+	)
 	(gr_text "."
 		(at 145.5 89.5 0)
@@
 		)
 	)
+	(gr_text "10"
+		(at 133.5 98.5 0)
+		(layer "F.SilkS")
+		(effects
+			(font
+				(size 1 1)
+				(thickness 0.1)
+			)
+			(justify left bottom)
+		)
+	)
 	(gr_text "."
 		(at 148.5 92.5 0)
@@
 		)
 	)
+	(gr_text "5"
+		(at 139.5 110 0)
+		(layer "F.SilkS")
+		(effects
+			(font
+				(size 1 1)
+				(thickness 0.1)
+			)
+			(justify left bottom)
+		)
+	)
 	(gr_text "."
 		(at 147 100 0)
@@
 		)
 	)
+	(gr_text "6"
+		(at 138.5 108 0)
+		(layer "F.SilkS")
+		(effects
+			(font
+				(size 1 1)
+				(thickness 0.1)
+			)
+			(justify left bottom)
+		)
+	)
 	(gr_text "."
 		(at 147 103 0)
@@
 		)
 	)
+	(gr_text "1"
+		(at 145.049295 120.65359 0)
+		(layer "F.SilkS")
+		(effects
+			(font
+				(size 1 1)
+				(thickness 0.1)
+			)
+			(justify left bottom)
+		)
+	)
 	(gr_text "."
 		(at 145.5 94 0)
@@
 		)
 	)
+	(gr_text "12"
+		(at 131.5 93.955821 0)
+		(layer "F.SilkS")
+		(effects
+			(font
+				(size 1 1)
+				(thickness 0.1)
+			)
+			(justify left bottom)
+		)
+	)
+	(gr_text "7"
+		(at 137.5 105.5 0)
+		(layer "F.SilkS")
+		(effects
+			(font
+				(size 1 1)
+				(thickness 0.1)
+			)
+			(justify left bottom)
+		)
+	)
 	(gr_text "."
 		(at 142.5 97 0)
@@
 		)
 	)
+	(gr_text "2"
+		(at 142 117 0)
+		(layer "F.SilkS")
+		(effects
+			(font
+				(size 1 1)
+				(thickness 0.1)
+			)
+			(justify left bottom)
+		)
+	)
 	(gr_text "."
 		(at 153 104.5 0)
@@
 		)
 	)
+	(gr_text "9"
+		(at 135.29943 100.5 0)
+		(layer "F.SilkS")
+		(effects
+			(font
+				(size 1 1)
+				(thickness 0.1)
+			)
+			(justify left bottom)
+		)
+	)
 	(gr_text "."
 		(at 145.5 100 0)
@@
 		)
 	)
+	(gr_text "12v"
+		(at 157.5 98 330)
+		(layer "F.SilkS")
+		(effects
+			(font
+				(size 1 1)
+				(thickness 0.1)
+				(italic yes)
+			)
+			(justify left bottom)
+		)
+	)
 	(gr_text "."
 		(at 142.5 98.5 0)
@@
 		)
 	)
+	(gr_text "4"
+		(at 141 112 0)
+		(layer "F.SilkS")
+		(effects
+			(font
+				(size 1 1)
+				(thickness 0.1)
+			)
+			(justify left bottom)
+		)
+	)
 	(gr_text "δ"
 		(at 139 94 0)
@@
 		)
 	)
+	(gr_text "3"
+		(at 141.5 114.5 0)
+		(layer "F.SilkS")
+		(effects
+			(font
+				(size 1 1)
+				(thickness 0.1)
+			)
+			(justify left bottom)
+		)
+	)
 	(gr_text "."
 		(at 147 92.5 0)
@@
 			)
 			(justify left bottom)
+		)
+	)
+	(gr_text "11"
+		(at 132.5 96 0)
+		(layer "F.SilkS")
+		(effects
+			(font
+				(size 1 1)
+				(thickness 0.1)
+			)
+			(justify left bottom)
