File: pcb/overview/overview.kicad_sch (KiCad schematic)
At the start: 13 parts, among them M1 Stepper_Motor_unipolar_6pin, M2 Stepper_Motor_unipolar_6pin, M3 Stepper_Motor_unipolar_6pin, M4 Motor_Servo, U1 ESP32-S3-DevKitC, U2 TCA9548APWR, U7 MPU-6050

Commit message: v0.4
Parts:
- added U10, U11, U9: ~, symbol main:LightBarrier
Connections:
- net at U1.21 (5V), U3.1 (VDD5V), U4.1 (VDD5V)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: now also U10.3 (5V), U11.3 (5V), U9.3 (5V)
- net at U1.22 (GND), U1.23 (GND), U1.24 (GND)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: now also U3.8 (DIR), U4.8 (DIR), U5.8 (DIR), U10.1 (GND), U11.1 (GND), U9.1 (GND)
- net at U1.14 (GPIO46): now also U9.2 (SIG)
- net at U1.16 (GPIO10/ADC1_CH9): now also U6.1 (EN1)
- net at U1.17 (GPIO11/ADC2_CH0): now also U6.2 (STEP1)
- net at U1.18 (GPIO12/ADC2_CH1): now also U6.3 (DIR1)
- net at U1.19 (GPIO13/ADC2_CH2): now also U6.4 (EN2)
- net at U1.20 (GPIO14/ADC2_CH3): now also U6.5 (STEP2)
- net at U1.27 (GPIO21): now also U6.6 (DIR2)
- net at U1.30 (GPIO45): now also U10.2 (SIG)
- net at U1.32 (GPIO35): now also U6.7 (EN3)
- net at U1.33 (GPIO36): now also U6.8 (STEP3)
- net at U1.34 (GPIO37): now also U6.9 (DIR3)
- net at U1.35 (GPIO38): now also U11.2 (SIG)
Other:
- moved on the sheet: M1, M2, M3, M4, R1, U2, U6, U7, U8
